File: hardware/hackboard/hackboard.kicad_pcb (KiCad board)
At the start: 2 copper layers, 22 parts, among them J1 Power, J2 Lil Cup, J3 Chonk Cup, J4 JTAG, Q1 30V 300mA, Q2 30V 300mA, U1 AP63200, U2 ESP32-WROVER-E

Commit message: PCB fertiggestellt
Parts:
- added J5: Programming Jumper, Connector_PinHeader_2.54mm:PinHeader_1x02_P2.54mm_Vertical, F.Cu at (160.0, 106.7)
- added REF**: MountingHole_3.2mm_M3_DIN965, MountingHole:MountingHole_3.2mm_M3_DIN965, F.Cu at (161.5, 115.3)
- added REF**: MountingHole_3.2mm_M3_DIN965, MountingHole:MountingHole_3.2mm_M3_DIN965, F.Cu at (161.5, 80.3)
- added REF**: MountingHole_3.2mm_M3_DIN965, MountingHole:MountingHole_3.2mm_M3_DIN965, F.Cu at (119.4, 80.3)
- added REF**: MountingHole_3.2mm_M3_DIN965, MountingHole:MountingHole_3.2mm_M3_DIN965, F.Cu at (119.4, 115.3)
- C3: footprint Capacitor_SMD:C_0603_1608Metric_Pad1.05x0.95mm_HandSolder -> Capacitor_SMD:C_0402_1005Metric
- J4: value JTAG -> Programming
- moved R1 66.3 mm to (120.4, 85.9), turned to 180 degrees
- moved C2 63.3 mm to (129.5, 90.4), turned to 90 degrees
- moved U1 52.4 mm to (125.5, 90.4)
- moved C3 51.7 mm to (120.4, 84.3), turned to 180 degrees
- moved R2 50.0 mm to (120.4, 87.4), turned to 180 degrees
- moved J4 36.1 mm to (161.0, 89.4), turned to 270 degrees
- moved J3 32.8 mm to (131.1, 104.6), turned to 270 degrees
- moved J2 15.3 mm to (122.4, 104.6), turned to 270 degrees
- moved L1 13.2 mm to (126.5, 83.8), turned to 180 degrees
- moved J1 12.5 mm to (122.4, 95.5), turned to 270 degrees
- moved Q1 9.54 mm to (130.6, 95.5)
- moved Q2 9.54 mm to (130.6, 99.6)
- moved R3 9.44 mm to (135.1, 95.6)
- moved R4 9.44 mm to (135.1, 99.6)
- moved C4 9.27 mm to (133.6, 80.8), turned to 0 degrees
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Connections:
- J4 pad 1: Net-(J4-Pad1) -> (no net)
- J4 pad 4: Net-(J4-Pad4) -> Vin
- J4 pad 5: (no net) -> +3V3
- J4 pad 6: (no net) -> GND
- U2 pad 10: Net-(U2-Pad10) -> (no net)
- U2 pad 11: Net-(U2-Pad11) -> (no net)
- U2 pad 12: Net-(U2-Pad12) -> (no net)
- U2 pad 13: Net-(J4-Pad1) -> (no net)
- U2 pad 14: Net-(J4-Pad2) -> (no net)
- U2 pad 16: Net-(J4-Pad3) -> (no net)
- U2 pad 17: Net-(U2-Pad17) -> (no net)
- U2 pad 18: Net-(U2-Pad18) -> (no net)
- U2 pad 19: Net-(U2-Pad19) -> (no net)
- U2 pad 20: Net-(U2-Pad20) -> (no net)
- U2 pad 21: Net-(U2-Pad21) -> (no net)
- U2 pad 22: Net-(U2-Pad22) -> (no net)
- U2 pad 23: Net-(J4-Pad4) -> (no net)
- U2 pad 24: Net-(U2-Pad24) -> (no net)
- U2 pad 26: Net-(U2-Pad26) -> (no net)
- U2 pad 27: Net-(U2-Pad27) -> (no net)
- U2 pad 28: Net-(U2-Pad28) -> (no net)
- U2 pad 29: Net-(U2-Pad29) -> (no net)
- U2 pad 30: Net-(U2-Pad30) -> (no net)
- U2 pad 31: Net-(U2-Pad31) -> (no net)
- U2 pad 32: Net-(U2-Pad32) -> (no net)
- U2 pad 33: Net-(U2-Pad33) -> (no net)
- U2 pad 34: Net-(U2-Pad34) -> Net-(J4-Pad3)
- U2 pad 35: Net-(U2-Pad35) -> Net-(J4-Pad2)
- U2 pad 36: Net-(U2-Pad36) -> (no net)
- U2 pad 37: Net-(U2-Pad37) -> (no net)
- U2 pad 4: Net-(U2-Pad4) -> (no net)
- U2 pad 5: Net-(U2-Pad5) -> (no net)
- U2 pad 8: Net-(U2-Pad8) -> (no net)
- U2 pad 9: Net-(U2-Pad9) -> (no net)
Routing:
- net +3V3: track 0.00 -> 69.4 mm, vias 0 -> 2
- net Vin: track 0.00 -> 52.8 mm, vias 0 -> 1
- net Drain1: track 0.00 -> 18.9 mm
- net Source1: track 0.00 -> 17.7 mm
- net Net-(C2-Pad1): track 0.00 -> 11.5 mm
- net Source2: track 0.00 -> 9.34 mm
- net Net-(C3-Pad2): track 0.00 -> 8.48 mm
- net Net-(C8-Pad1): track 0.00 -> 8.12 mm
- net Drain2: track 0.00 -> 7.56 mm
- net Net-(J4-Pad3): track 0.00 -> 6.25 mm
- net Net-(J4-Pad2): track 0.00 -> 6.24 mm
- net Net-(J5-Pad1): track 0.00 -> 5.55 mm
- net Net-(R4-Pad1): track 0.00 -> 4.68 mm
- net Net-(Q2-Pad1): track 0.00 -> 3.10 mm
- net Net-(Q1-Pad1): track 0.00 -> 3.10 mm
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- added copper zone on B.Cu, net GND
- added copper zone on F.Cu, net GND
Other:
- board outline added: 52.3 x 45.2 mm
- board text added: "2022 - Fjore & Lytrox"
- board text added: "Smartbrain moves for NespressOwO machines!"
